Commit message: URDF- remove unnecessary collision sections - resulted to weird convex visualization on rviz

File: urdf/go1.urdf (robot description, URDF)
Before this commit: robot mc_go1_description, 46 links, 45 joints
Links:
- link FL_calf_rotor: geometry visual cylinder length=0.02 radius=0.035
- link FL_foot: geometry visual sphere radius=0.01
- link FL_hip_rotor: geometry visual cylinder length=0.02 radius=0.035
- link FL_thigh_rotor: geometry visual cylinder length=0.02 radius=0.035
- link FR_calf_rotor: geometry visual cylinder length=0.02 radius=0.035
- link FR_foot: geometry visual sphere radius=0.01
- link FR_hip_rotor: geometry visual cylinder length=0.02 radius=0.035
- link FR_thigh_rotor: geometry visual cylinder length=0.02 radius=0.035
- link RL_calf_rotor: geometry visual cylinder length=0.02 radius=0.035
- link RL_foot: geometry visual sphere radius=0.01
- link RL_hip_rotor: geometry visual cylinder length=0.02 radius=0.035
- link RL_thigh_rotor: geometry visual cylinder length=0.02 radius=0.035
- link RR_calf_rotor: geometry visual cylinder length=0.02 radius=0.035
- link RR_foot: geometry visual sphere radius=0.01
- link RR_hip_rotor: geometry visual cylinder length=0.02 radius=0.035
- link RR_thigh_rotor: geometry visual cylinder length=0.02 radius=0.035
